Commit message: correctly attach base_link and camera_mount_plate by applying offsets
instead of putting them in each other

File: airo_models/grippers/schunk_egk40_magneto/schunk_egk40_magneto.urdf (robot description, URDF)
Before this commit: robot schunk_egk40_magneto, 8 links, 7 joints
Joints:
- joint base_link_gripper_joint: origin (none) -> xyz=0 0 0.00175
- joint base_link_to_camera_mount_plate: origin (none) -> xyz=0 0 0.00925
